Commit message: refactoring description package and created a gazebo_package

File: urdf/lidar_sensor.xacro (robot description, xacro)
@@ -64,36 +64,36 @@
     <gazebo reference="hokuyo">
     </gazebo>
-  <gazebo reference="hokuyo_lidar">
-    <sensor type="ray" name="hokuyo_lidar_sensor">
-      <always_on>true</always_on>
-      <pose relative_to="hokuyo_lidar">0 0 0 0 0 0</pose>
-      <visualize>false</visualize>
-      <update_rate>20</update_rate>
-      <ray>
-        <scan>
-          <horizontal>
-            <samples>720</samples>
-            <resolution>1</resolution>
-            <min_angle>-3.14</min_angle>
-            <max_angle>3.14</max_angle>
-          </horizontal>
-        </scan>
-        <range>
-          <min>0.5</min>
-          <max>20</max>
-          <resolution>0.01</resolution>
-        </range>
-        <noise>
-          <type>gaussian</type>
-          <mean>0.0</mean>
-          <stddev>0.01</stddev>
-        </noise>
-      </ray>
-      <plugin name="lidar" filename="libgazebo_ros_laser.so">
-        <output_type>sensor_msgs/LaserScan</output_type>
-        <frameName>hokuyo_lidar</frameName>
-        <topicName>/scan</topicName>
-      </plugin>
-    </sensor>
-  </gazebo>
+    <gazebo reference="hokuyo_lidar">
+      <sensor type="ray" name="hokuyo_lidar_sensor">
+        <always_on>true</always_on>
+        <pose relative_to="hokuyo_lidar">0 0 0 0 0 0</pose>
+        <visualize>false</visualize>
+        <update_rate>20</update_rate>
+        <ray>
+          <scan>
+            <horizontal>
+              <samples>720</samples>
+              <resolution>1</resolution>
+              <min_angle>-3.14</min_angle>
+              <max_angle>3.14</max_angle>
+            </horizontal>
+          </scan>
+          <range>
+            <min>0.5</min>
+            <max>20</max>
+            <resolution>0.01</resolution>
+          </range>
+          <noise>
+            <type>gaussian</type>
+            <mean>0.0</mean>
+            <stddev>0.01</stddev>
+          </noise>
+        </ray>
+        <plugin name="lidar" filename="libgazebo_ros_laser.so">
+          <output_type>sensor_msgs/LaserScan</output_type>
+          <frameName>hokuyo_lidar</frameName>
+          <topicName>/scan</topicName>
+        </plugin>
+      </sensor>
+    </gazebo>
 </robot>

File: urdf/my_robot_assembly.xacro (robot description, xacro)
@@ -5,4 +5,6 @@
     <!-- importing the template for the robot wheels -->
     <xacro:include filename="$(find my_robot_description)/urdf/my_wheel.xacro"/>
+    <!-- importing all the related gazebo configurations -->
+    <!-- <xacro:include filename="$(find my_robot_description)/urdf/gazebo.xacro"/> -->
     <!-- Macros for importing the lidar -->
     <xacro:include filename="$(find my_robot_description)/urdf/lidar_sensor.xacro"/>

File: urdf/my_wheel.xacro (robot description, xacro)
@@ -21,4 +21,5 @@
         </inertial>
     </xacro:macro>
+    <!-- </xacro:property> -->
 <!-- creating a xacro macro for the template of the wheels -->
     <xacro:macro name="wheel" params="name x y file_path">
@@ -87,3 +88,27 @@
         </plugin>
     </gazebo>
+    <xacro:macro name="transmission_macro" params="name joint_name actuator_name">
+        <transmission name="${name}" >
+            <type>transmission_interface/SimpleTransmission</type>
+            <joint name="${joint_name}">
+                <hardwareInterface>hardware_interface/EffortJointInterface</hardwareInterface>
+            </joint>
+            <actuator name="${actuator_name}">
+                <hardwareInterface>hardware_interface/EffortJointInterface</hardwareInterface>
+                <mechanicalReduction>1</mechanicalReduction>
+            </actuator>
+        </transmission>
+    </xacro:macro>
+    <!-- creating the transmissions for each joint  -->
+    <xacro:transmission_macro name="rear_right_transmission" joint_name="wheel_rear_right_joint" actuator_name="dc_motor_rr" />
+    <xacro:transmission_macro name="rear_left_transmission" joint_name="wheel_rear_left_joint" actuator_name="dc_motor_ll" />
+    <xacro:transmission_macro name="front_right_transmission" joint_name="wheel_front_right_joint" actuator_name="dc_motor_fr" />
+    <xacro:transmission_macro name="front_left_transmission" joint_name="wheel_front_left_joint" actuator_name="dc_motor_fl" />
+    <!-- adding the ros control plugin: It creates a communication between the comand from a controller
+    to the joints -->
+    <gazebo>
+        <plugin name="gazebo_ros_control" filename="libgazebo_ros_control.so">
+            <robotNamespace>/my_robot</robotNamespace>
+        </plugin>
+    </gazebo>
 </robot>
