Commit message: modified to use skid_steer plugin for simple teleop

File: urdf/my_wheel.xacro (robot description, xacro)
@@ -73,5 +73,5 @@
             <wheelSeparation>0.8</wheelSeparation>
             <wheelDiameter>${2 * wheel_radius}</wheelDiameter>
-            <robotBaseFrame>base_footprint</robotBaseFrame>
+            <robotBaseFrame>base_link</robotBaseFrame>
             <torque>50</torque>
             <!-- for sending command messages (twist) -->
@@ -88,27 +88,27 @@
         </plugin>
     </gazebo>
-    <xacro:macro name="transmission_macro" params="name joint_name actuator_name">
+    <!-- <xacro:macro name="transmission_macro" params="name joint_name actuator_name">
         <transmission name="${name}" >
             <type>transmission_interface/SimpleTransmission</type>
             <joint name="${joint_name}">
-                <hardwareInterface>hardware_interface/EffortJointInterface</hardwareInterface>
+                <hardwareInterface>hardware_interface/VelocityJointInterface</hardwareInterface>
             </joint>
             <actuator name="${actuator_name}">
-                <hardwareInterface>hardware_interface/EffortJointInterface</hardwareInterface>
+                <hardwareInterface>hardware_interface/VelocityJointInterface</hardwareInterface>
                 <mechanicalReduction>1</mechanicalReduction>
             </actuator>
         </transmission>
-    </xacro:macro>
+    </xacro:macro> -->
     <!-- creating the transmissions for each joint  -->
-    <xacro:transmission_macro name="rear_right_transmission" joint_name="wheel_rear_right_joint" actuator_name="dc_motor_rr" />
+    <!-- <xacro:transmission_macro name="rear_right_transmission" joint_name="wheel_rear_right_joint" actuator_name="dc_motor_rr" />
     <xacro:transmission_macro name="rear_left_transmission" joint_name="wheel_rear_left_joint" actuator_name="dc_motor_ll" />
     <xacro:transmission_macro name="front_right_transmission" joint_name="wheel_front_right_joint" actuator_name="dc_motor_fr" />
-    <xacro:transmission_macro name="front_left_transmission" joint_name="wheel_front_left_joint" actuator_name="dc_motor_fl" />
+    <xacro:transmission_macro name="front_left_transmission" joint_name="wheel_front_left_joint" actuator_name="dc_motor_fl" /> -->
     <!-- adding the ros control plugin: It creates a communication between the comand from a controller
     to the joints -->
-    <gazebo>
+    <!-- <gazebo>
         <plugin name="gazebo_ros_control" filename="libgazebo_ros_control.so">
             <robotNamespace>/my_robot</robotNamespace>
         </plugin>
-    </gazebo>
+    </gazebo> -->
 </robot>
